File: CartGen4/spi.kicad_sch (KiCad schematic)
At the start: 11 parts, among them J1 MEM2080-00-128-00-A, U10 IS25WP080D-JNLE, U11 DS1391U-33+, Y1 FC-135R_32.7680KA-E5

Commit message: Cleaned up symbol fields
Parts:
- U11: Datasheet_1 https://componentsearchengine.com/Datasheets/2/DS1391U-33+.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 -> (none); Footprint_1 SOP50P490X110-10N -> (none); Height 1.1 -> (none); MFN (none) -> Analog Devices; MFP (none) -> DS1391U-33+; Manufacturer_Name Analog Devices -> (none); Manufacturer_Part_Number DS1391U-33+ -> (none); Mouser Part Number 700-DS1391U-33 -> (none); Mouser Price/Stock https://www.mouser.co.uk/ProductDetail/Analog-Devices-Maxim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 -> (none); Reference_1 IC -> (none); Value_1 DS1391U-33+ -> (none)
- Y1: Datasheet_1 https://support.epson.biz/td/api/doc_check.php?dl=brief_FC-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 -> (none); Footprint_1 FC135R327680KAE3 -> (none); Height 0.9 -> (none); MFN (none) -> Epson Timing; MFP (none) -> FC-135R 32.7680KA-E3; Manufacturer_Name Epson Timing -> (none); Manufacturer_Part_Number FC-135R 32.7680KA-E3 -> (none); Mouser Part Number 732-5R32.7680KA-E3 -> (none); Mouser Price/Stock https://www.mouser.co.uk/ProductDetail/Epson-Timing/FC-135R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 -> (none); Reference_1 Y -> (none); Value_1 FC-135R_32.7680KA-E3 -> (none)
Changed lines of the file:
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@@
       (effects (font (size 1.27 1.27)) hide)
     )
-    (property "Datasheet" "" (id 3) (at 176.53 68.58 0)
+    (property "Datasheet" "https://eu.mouser.com/datasheet/2/137/FC_255_en-1649561.pdf" (id 3) (at 176.53 68.58 0)
       (effects (font (size 1.27 1.27)) hide)
     )
-    (property "Reference_1" "Y" (id 4) (at 161.29 64.77 0)
+    (property "MFN" "Epson Timing" (id 11) (at 872.72 59.69 0)
       (effects (font (size 1.27 1.27)) (justify left top) hide)
     )
-    (property "Value_1" "FC-135R_32.7680KA-E3" (id 5) (at 163.83 74.93 0)
-      (effects (font (size 1.27 1.27)) (justify left top) hide)
-    )
-    (property "Footprint_1" "FC135R327680KAE3" (id 6) (at 272.72 59.69 0)
-      (effects (font (size 1.27 1.27)) (justify left top) hide)
-    )
-    (property "Datasheet_1" "https://support.epson.biz/td/api/doc_check.php?dl=brief_FC-135R&lang=en" (id 7) (at 372.72 59.69 0)
-      (effects (font (size 1.27 1.27)) (justify left top) hide)
-    )
-    (property "Height" "0.9" (id 8) (at 572.72 59.69 0)
-      (effects (font (size 1.27 1.27)) (justify left top) hide)
-    )
-    (property "Mouser Part Number" "732-5R32.7680KA-E3" (id 9) (at 672.72 59.69 0)
-      (effects (font (size 1.27 1.27)) (justify left top) hide)
-    )
-    (property "Mouser Price/Stock" "https://www.mouser.co.uk/ProductDetail/Epson-Timing/FC-135R-32.7680KA-E3?qs=f9yNj16SXrI2dPFQj6LACQ%3D%3D" (id 10) (at 772.72 59.69 0)
-      (effects (font (size 1.27 1.27)) (justify left top) hide)
-    )
-    (property "Manufacturer_Name" "Epson Timing" (id 11) (at 872.72 59.69 0)
-      (effects (font (size 1.27 1.27)) (justify left top) hide)
-    )
-    (property "Manufacturer_Part_Number" "FC-135R 32.7680KA-E3" (id 12) (at 972.72 59.69 0)
+    (property "MFP" "FC-135R 32.7680KA-E3" (id 12) (at 972.72 59.69 0)
       (effects (font (size 1.27 1.27)) (justify left top) hide)
     )
@@
       (effects (font (size 1.27 1.27)) hide)
     )
-    (property "Datasheet" "https://nl.mouser.com/datasheet/2/609/DS1390_DS1394-3122080.pdf" (id 3) (at 194.31 68.58 0)
+    (property "Datasheet" "https://eu.mouser.com/datasheet/2/609/DS1390_DS1394-3122080.pdf" (id 3) (at 194.31 68.58 0)
       (effects (font (size 1.27 1.27)) hide)
     )
-    (property "Reference_1" "IC" (id 4) (at 210.82 55.88 0)
-      (effects (font (size 1.27 1.27)) hide)
-    )
-    (property "Value_1" "DS1391U-33+" (id 5) (at 210.82 58.42 0)
-      (effects (font (size 1.27 1.27)) hide)
-    )
-    (property "Footprint_1" "SOP50P490X110-10N" (id 6) (at 223.52 163.5 0)
+    (property "MFN" "Analog Devices" (id 4) (at 223.52 763.5 0)
       (effects (font (size 1.27 1.27)) (justify left top) hide)
     )
-    (property "Datasheet_1" "https://componentsearchengine.com/Datasheets/2/DS1391U-33+.pdf" (id 7) (at 223.52 263.5 0)
+    (property "MFP" "DS1391U-33+" (id 5) (at 223.52 863.5 0)
       (effects (font (size 1.27 1.27)) (justify left top) hide)
     )
-    (property "Height" "1.1" (id 8) (at 223.52 463.5 0)
-      (effects (font (size 1.27 1.27)) (justify left top) hide)
-    )
-    (property "Mouser Part Number" "700-DS1391U-33" (id 9) (at 223.52 563.5 0)
-      (effects (font (size 1.27 1.27)) (justify left top) hide)
-    )
-    (property "Mouser Price/Stock" "https://www.mouser.co.uk/ProductDetail/Analog-Devices-Maxim-Integrated/DS1391U-33%2b?qs=0Y9aZN%252BMVCVmg1eZRkyk7Q%3D%3D" (id 10) (at 223.52 663.5 0)
-      (effects (font (size 1.27 1.27)) (justify left top) hide)
-    )
-    (property "Manufacturer_Name" "Analog Devices" (id 11) (at 223.52 763.5 0)
-      (effects (font (size 1.27 1.27)) (justify left top) hide)
-    )
-    (property "Manufacturer_Part_Number" "DS1391U-33+" (id 12) (at 223.52 863.5 0)
-      (effects (font (size 1.27 1.27)) (justify left top) hide)
-    )

Commit message: Added symbol information to obvious stuff
Parts:
- BT1: Critical (none) -> N; Notes (none) -> Battery is utilised and maintained by the DS1391U-33+ RTC.
- C33, C34, C35: Critical (none) -> N; Notes (none) -> Bypass capacitor for PWR/GND coupling.
- J1: Critical (none) -> Y; MFN (none) -> GCT; MFP (none) -> MEM2080-00-128-00-A
- U10: Critical (none) -> Y; MFN (none) -> ISSI; MFP (none) -> IS25WP080D-JNLE; Notes (none) -> Used for storing FPGA configuration and boot code.; Package ID (none) -> SOIC-8; Source (none) -> SPEC
- U11: Critical (none) -> N; Notes (none) -> RTC for timekeeping functions.; Package ID (none) -> MSOP-10; Source (none) -> SPEC
- Y1: Critical (none) -> N; Notes (none) -> Crystal for RTC clock.; Source (none) -> SPEC
Changed lines of the file:
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@@
       (effects (font (size 1.27 1.27)) hide)
     )
-    (property "Datasheet" "" (id 3) (at 87.63 148.59 0)
+    (property "Datasheet" "https://eu.mouser.com/datasheet/2/837/Global_Connector_gct_mem2080_npi_flyer_V1_0-3007328.pdf" (id 3) (at 87.63 148.59 0)
+      (effects (font (size 1.27 1.27)) hide)
+    )
+    (property "Critical" "Y" (id 4) (at 87.63 132.08 0)
+      (effects (font (size 1.27 1.27)) hide)
+    )
+    (property "Description" "Memory Card Connectors Micro SD, Push Push, SMT, Card Entry Normal, 1.28 mm profile" (id 5) (at 87.63 132.08 0)
+      (effects (font (size 1.27 1.27)) hide)
+    )
+    (property "MFN" "GCT" (id 6) (at 87.63 132.08 0)
+      (effects (font (size 1.27 1.27)) hide)
+    )
+    (property "MFP" "MEM2080-00-128-00-A" (id 7) (at 87.63 132.08 0)
       (effects (font (size 1.27 1.27)) hide)
     )
@@
       (effects (font (size 1.27 1.27)) hide)
     )
+    (property "Critical" "N" (id 4) (at 118.11 76.2 0)
+      (effects (font (size 1.27 1.27)) hide)
+    )
+    (property "Notes" "Bypass capacitor for PWR/GND coupling." (id 5) (at 118.11 76.2 0)
+      (effects (font (size 1.27 1.27)) hide)
+    )
     (pin "1")
     (pin "2")
@@
     )
     (property "Datasheet" "~" (id 3) (at 58.42 132.08 0)
+      (effects (font (size 1.27 1.27)) hide)
+    )
+    (property "Critical" "N" (id 4) (at 58.42 132.08 0)
+      (effects (font (size 1.27 1.27)) hide)
+    )
+    (property "Notes" "Bypass capacitor for PWR/GND coupling." (id 5) (at 58.42 132.08 0)
       (effects (font (size 1.27 1.27)) hide)
     )
@@
       (effects (font (size 1.27 1.27)) (justify left top) hide)
     )
+    (property "Description" "Crystals FC-135R 32.7680KA-E5: SMD XTL KHZ +/-20PPM,-40-85C 6.0PF 3K TR" (id 13) (at 176.53 68.58 0)
+      (effects (font (size 1.27 1.27)) hide)
+    )
+    (property "Notes" "Crystal for RTC clock." (id 14) (at 176.53 68.58 0)
+      (effects (font (size 1.27 1.27)) hide)
+    )
+    (property "Package ID" "~" (id 15) (at 176.53 68.58 0)
+      (effects (font (size 1.27 1.27)) hide)
+    )
+    (property "Source" "SPEC" (id 16) (at 176.53 68.58 0)
+      (effects (font (size 1.27 1.27)) hide)
+    )
+    (property "Critical" "N" (id 17) (at 176.53 68.58 0)
+      (effects (font (size 1.27 1.27)) hide)
+    )
     (pin "")
     (pin "2")
@@
     )
     (property "Datasheet" "~" (id 3) (at 252.73 74.93 0)
+      (effects (font (size 1.27 1.27)) hide)
+    )
+    (property "Critical" "N" (id 4) (at 252.73 74.93 0)
+      (effects (font (size 1.27 1.27)) hide)
+    )
+    (property "Notes" "Bypass capacitor for PWR/GND coupling." (id 5) (at 252.73 74.93 0)
       (effects (font (size 1.27 1.27)) hide)
     )
@@
       (effects (font (size 1.27 1.27)) hide)
     )
-    (property "Datasheet" "" (id 3) (at 67.31 69.85 0)
+    (property "Datasheet" "https://eu.mouser.com/datasheet/2/198/25LP_WP080D_040D_020D-1770149.pdf" (id 3) (at 67.31 69.85 0)
+      (effects (font (size 1.27 1.27)) hide)
+    )
+    (property "Critical" "Y" (id 4) (at 67.31 69.85 0)
+      (effects (font (size 1.27 1.27)) hide)
+    )
+    (property "Description" "NOR Flash 8M QSPI, 8-pin SOP 105mil ET" (id 5) (at 67.31 69.85 0)
+      (effects (font (size 1.27 1.27)) hide)
+    )
+    (property "MFN" "ISSI" (id 6) (at 67.31 69.85 0)
+      (effects (font (size 1.27 1.27)) hide)
+    )
+    (property "MFP" "IS25WP080D-JNLE" (id 7) (at 67.31 69.85 0)
+      (effects (font (size 1.27 1.27)) hide)
+    )
+    (property "Notes" "Used for storing FPGA configuration and boot code." (id 8) (at 67.31 69.85 0)
+      (effects (font (size 1.27 1.27)) hide)
+    )
+    (property "Source" "SPEC" (id 9) (at 67.31 69.85 0)
+      (effects (font (size 1.27 1.27)) hide)
+    )
+    (property "Package ID" "SOIC-8" (id 10) (at 67.31 69.85 0)
       (effects (font (size 1.27 1.27)) hide)
     )
@@
     (property "MFP" "DS1391U-33+" (id 5) (at 223.52 863.5 0)
       (effects (font (size 1.27 1.27)) (justify left top) hide)
+    )
+    (property "Critical" "N" (id 6) (at 194.31 68.58 0)
+      (effects (font (size 1.27 1.27)) hide)
+    )
+    (property "Description" "Real Time Clock Low-Voltage SPI/3-Wire RTCs with Trickle Charger" (id 7) (at 194.31 68.58 0)
+      (effects (font (size 1.27 1.27)) hide)
+    )
+    (property "Notes" "RTC for timekeeping functions." (id 8) (at 194.31 68.58 0)
+      (effects (font (size 1.27 1.27)) hide)
+    )
+    (property "Package ID" "MSOP-10" (id 9) (at 194.31 68.58 0)
+      (effects (font (size 1.27 1.27)) hide)
+    )
+    (property "Source" "SPEC" (id 10) (at 194.31 68.58 0)
+      (effects (font (size 1.27 1.27)) hide)
     )
     (pin "1")
@@
       (effects (font (size 1.27 1.27)) hide)
     )
+    (property "Critical" "N" (id 4) (at 184.15 95.25 0)
+      (effects (font (size 1.27 1.27)) hide)
+    )
+    (property "Notes" "Battery is utilised and maintained by the DS1391U-33+ RTC." (id 5) (at 184.15 95.25 0)
+      (effects (font (size 1.27 1.27)) hide)
+    )

Commit message: Added more symbol information
Parts:
- BT1: Source (none) -> SPEC
- C33, C34, C35: Source (none) -> ANY
- R16, R17, R18: Critical (none) -> Y; Source (none) -> ANY; Tolerance (none) -> 10%
Changed lines of the file:
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@@
+      (effects (font (size 1.27 1.27)) hide)
+    )
+    (property "Tolerance" "10%" (id 4) (at 167.64 69.85 0)
+      (effects (font (size 1.27 1.27)) hide)
+    )
+    (property "Source" "ANY" (id 5) (at 167.64 69.85 0)
+      (effects (font (size 1.27 1.27)) hide)
+    )
+    (property "Critical" "Y" (id 6) (at 167.64 69.85 0)
       (effects (font (size 1.27 1.27)) hide)
     )
@@
       (effects (font (size 1.27 1.27)) hide)
     )
+    (property "Source" "ANY" (id 6) (at 118.11 76.2 0)
+      (effects (font (size 1.27 1.27)) hide)
+    )
     (pin "1")
     (pin "2")
@@
     )
     (property "Notes" "Bypass capacitor for PWR/GND coupling." (id 5) (at 58.42 132.08 0)
+      (effects (font (size 1.27 1.27)) hide)
+    )
+    (property "Source" "ANY" (id 6) (at 58.42 132.08 0)
       (effects (font (size 1.27 1.27)) hide)
     )
@@
       (effects (font (size 1.27 1.27)) hide)
     )
+    (property "Tolerance" "10%" (id 4) (at 45.72 139.7 0)
+      (effects (font (size 1.27 1.27)) hide)
+    )
+    (property "Source" "ANY" (id 5) (at 45.72 139.7 0)
+      (effects (font (size 1.27 1.27)) hide)
+    )
+    (property "Critical" "Y" (id 6) (at 45.72 139.7 0)
+      (effects (font (size 1.27 1.27)) hide)
+    )
     (pin "1")
     (pin "2")
@@
     )
     (property "Notes" "Bypass capacitor for PWR/GND coupling." (id 5) (at 252.73 74.93 0)
+      (effects (font (size 1.27 1.27)) hide)
+    )
+    (property "Source" "ANY" (id 6) (at 252.73 74.93 0)
       (effects (font (size 1.27 1.27)) hide)
     )
@@
       (effects (font (size 1.27 1.27)) hide)
     )
+    (property "Source" "SPEC" (id 6) (at 184.15 95.25 0)
+      (effects (font (size 1.27 1.27)) hide)
+    )
     (pin "1")
     (pin "2")
@@
       (effects (font (size 1.27 1.27)) hide)
     )
+    (property "Tolerance" "10%" (id 4) (at 54.61 63.5 0)
+      (effects (font (size 1.27 1.27)) hide)
+    )
+    (property "Source" "ANY" (id 5) (at 54.61 63.5 0)
+      (effects (font (size 1.27 1.27)) hide)
+    )
+    (property "Critical" "Y" (id 6) (at 54.61 63.5 0)
+      (effects (font (size 1.27 1.27)) hide)
+    )
