File: CartGen4/fpga_0.kicad_sch (KiCad schematic)
At the start: 12 parts, among them U9 LFXP2-8E-5MN132C

Commit message: Added symbol information to obvious stuff
Parts:
- C19, C20, C21, C22, C23, C24, C25, C30, C31, C32: Critical (none) -> N; Notes (none) -> Bypass capacitor for PWR/GND coupling.
- U9: Critical (none) -> Y; MFN (none) -> Lattice; MFP (none) -> LFXP2-8E-5MN132C; Notes (none) -> FPGA used for the bulk of the cartridge's functions (MBC em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; Package ID (none) -> CSBGA-132; Source (none) -> SPEC
Changed lines of the file:
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@@
+      (effects (font (size 1.27 1.27)) hide)
+    )
+    (property "Critical" "N" (id 4) (at 204.47 29.21 0)
+      (effects (font (size 1.27 1.27)) hide)
+    )
+    (property "Notes" "Bypass capacitor for PWR/GND coupling." (id 5) (at 204.47 29.21 0)
       (effects (font (size 1.27 1.27)) hide)
     )
@@
       (effects (font (size 1.27 1.27)) hide)
     )
-    (property "Datasheet" "" (id 3) (at 101.6 121.92 0)
+    (property "Datasheet" "https://www.latticesemi.com/view_document?document_id=24635" (id 3) (at 101.6 121.92 0)
+      (effects (font (size 1.27 1.27)) hide)
+    )
+    (property "Critical" "Y" (id 4) (at 97.79 124.46 0)
+      (effects (font (size 1.27 1.27)) hide)
+    )
+    (property "Description" "FPGA - Field Programmable Gate Array 8K LUTs 86I/O Inst- on DSP 1.2V -5 Spd" (id 5) (at 97.79 124.46 0)
+      (effects (font (size 1.27 1.27)) hide)
+    )
+    (property "MFN" "Lattice" (id 6) (at 97.79 124.46 0)
+      (effects (font (size 1.27 1.27)) hide)
+    )
+    (property "MFP" "LFXP2-8E-5MN132C" (id 7) (at 97.79 124.46 0)
+      (effects (font (size 1.27 1.27)) hide)
+    )
+    (property "Notes" "FPGA used for the bulk of the cartridge's functions (MBC emulation, SPI bridge, MMU functions, etc.)." (id 8) (at 97.79 124.46 0)
+      (effects (font (size 1.27 1.27)) hide)
+    )
+    (property "Package ID" "CSBGA-132" (id 9) (at 97.79 124.46 0)
+      (effects (font (size 1.27 1.27)) hide)
+    )
+    (property "Source" "SPEC" (id 10) (at 97.79 124.46 0)
       (effects (font (size 1.27 1.27)) hide)
     )
@@
       (effects (font (size 1.27 1.27)) hide)
     )
-    (property "Datasheet" "" (id 3) (at 62.23 41.91 0)
+    (property "Datasheet" "https://www.latticesemi.com/view_document?document_id=24635" (id 3) (at 62.23 41.91 0)
+      (effects (font (size 1.27 1.27)) hide)
+    )
+    (property "Critical" "Y" (id 4) (at 58.42 44.45 0)
+      (effects (font (size 1.27 1.27)) hide)
+    )
+    (property "Description" "FPGA - Field Programmable Gate Array 8K LUTs 86I/O Inst- on DSP 1.2V -5 Spd" (id 5) (at 58.42 44.45 0)
+      (effects (font (size 1.27 1.27)) hide)
+    )
+    (property "MFN" "Lattice" (id 6) (at 58.42 44.45 0)
+      (effects (font (size 1.27 1.27)) hide)
+    )
+    (property "MFP" "LFXP2-8E-5MN132C" (id 7) (at 58.42 44.45 0)
+      (effects (font (size 1.27 1.27)) hide)
+    )
+    (property "Notes" "FPGA used for the bulk of the cartridge's functions (MBC emulation, SPI bridge, MMU functions, etc.)." (id 8) (at 58.42 44.45 0)
+      (effects (font (size 1.27 1.27)) hide)
+    )
+    (property "Package ID" "CSBGA-132" (id 9) (at 58.42 44.45 0)
+      (effects (font (size 1.27 1.27)) hide)
+    )
+    (property "Source" "SPEC" (id 10) (at 58.42 44.45 0)
       (effects (font (size 1.27 1.27)) hide)
     )
@@
       (effects (font (size 1.27 1.27)) hide)
     )
-    (property "Datasheet" "" (id 3) (at 152.4 25.4 0)
+    (property "Datasheet" "https://www.latticesemi.com/view_document?document_id=24635" (id 3) (at 152.4 25.4 0)
+      (effects (font (size 1.27 1.27)) hide)
+    )
+    (property "Critical" "Y" (id 4) (at 148.59 27.94 0)
+      (effects (font (size 1.27 1.27)) hide)
+    )
+    (property "Description" "FPGA - Field Programmable Gate Array 8K LUTs 86I/O Inst- on DSP 1.2V -5 Spd" (id 5) (at 148.59 27.94 0)
+      (effects (font (size 1.27 1.27)) hide)
+    )
+    (property "MFN" "Lattice" (id 6) (at 148.59 27.94 0)
+      (effects (font (size 1.27 1.27)) hide)
+    )
+    (property "MFP" "LFXP2-8E-5MN132C" (id 7) (at 148.59 27.94 0)
+      (effects (font (size 1.27 1.27)) hide)
+    )
+    (property "Notes" "FPGA used for the bulk of the cartridge's functions (MBC emulation, SPI bridge, MMU functions, etc.)." (id 8) (at 148.59 27.94 0)
+      (effects (font (size 1.27 1.27)) hide)
+    )
+    (property "Package ID" "CSBGA-132" (id 9) (at 148.59 27.94 0)
+      (effects (font (size 1.27 1.27)) hide)
+    )
+    (property "Source" "SPEC" (id 10) (at 148.59 27.94 0)
       (effects (font (size 1.27 1.27)) hide)
     )
@@
       (effects (font (size 1.27 1.27)) hide)
     )
+    (property "Critical" "N" (id 4) (at 39.37 156.21 0)
+      (effects (font (size 1.27 1.27)) hide)
+    )
+    (property "Notes" "Bypass capacitor for PWR/GND coupling." (id 5) (at 39.37 156.21 0)
+      (effects (font (size 1.27 1.27)) hide)
+    )
     (pin "1")
     (pin "2")
@@
       (effects (font (size 1.27 1.27)) hide)
     )
+    (property "Critical" "N" (id 4) (at 116.84 36.83 0)
+      (effects (font (size 1.27 1.27)) hide)
+    )
+    (property "Notes" "Bypass capacitor for PWR/GND coupling." (id 5) (at 116.84 36.83 0)
+      (effects (font (size 1.27 1.27)) hide)
+    )
     (pin "1")
     (pin "2")
@@
       (effects (font (size 1.27 1.27)) hide)
     )
+    (property "Critical" "N" (id 4) (at 180.34 134.62 0)
+      (effects (font (size 1.27 1.27)) hide)
+    )
+    (property "Notes" "Bypass capacitor for PWR/GND coupling." (id 5) (at 180.34 134.62 0)
+      (effects (font (size 1.27 1.27)) hide)
+    )
     (pin "1")
     (pin "2")
@@
     )
     (property "Datasheet" "~" (id 3) (at 64.77 133.35 0)
+      (effects (font (size 1.27 1.27)) hide)
+    )
+    (property "Critical" "N" (id 4) (at 64.77 133.35 0)
+      (effects (font (size 1.27 1.27)) hide)
+    )
+    (property "Notes" "Bypass capacitor for PWR/GND coupling." (id 5) (at 64.77 133.35 0)
       (effects (font (size 1.27 1.27)) hide)
     )
@@
       (effects (font (size 1.27 1.27)) hide)
     )
-    (property "Datasheet" "" (id 3) (at 218.44 123.19 0)
+    (property "Datasheet" "https://www.latticesemi.com/view_document?document_id=24635" (id 3) (at 218.44 123.19 0)
+      (effects (font (size 1.27 1.27)) hide)
+    )
+    (property "Critical" "Y" (id 4) (at 214.63 125.73 0)
+      (effects (font (size 1.27 1.27)) hide)
+    )
+    (property "Description" "FPGA - Field Programmable Gate Array 8K LUTs 86I/O Inst- on DSP 1.2V -5 Spd" (id 5) (at 214.63 125.73 0)
+      (effects (font (size 1.27 1.27)) hide)
+    )
+    (property "MFN" "Lattice" (id 6) (at 214.63 125.73 0)
+      (effects (font (size 1.27 1.27)) hide)
+    )
+    (property "MFP" "LFXP2-8E-5MN132C" (id 7) (at 214.63 125.73 0)
+      (effects (font (size 1.27 1.27)) hide)
+    )
+    (property "Notes" "FPGA used for the bulk of the cartridge's functions (MBC emulation, SPI bridge, MMU functions, etc.)." (id 8) (at 214.63 125.73 0)
+      (effects (font (size 1.27 1.27)) hide)
+    )
+    (property "Package ID" "CSBGA-132" (id 9) (at 214.63 125.73 0)
+      (effects (font (size 1.27 1.27)) hide)
+    )
+    (property "Source" "SPEC" (id 10) (at 214.63 125.73 0)
       (effects (font (size 1.27 1.27)) hide)
     )
@@
       (effects (font (size 1.27 1.27)) hide)
     )
+    (property "Critical" "N" (id 4) (at 52.07 133.35 0)
+      (effects (font (size 1.27 1.27)) hide)
+    )
+    (property "Notes" "Bypass capacitor for PWR/GND coupling." (id 5) (at 52.07 133.35 0)
+      (effects (font (size 1.27 1.27)) hide)
+    )
     (pin "1")
     (pin "2")
@@
     )
     (property "Datasheet" "~" (id 3) (at 26.67 53.34 0)
+      (effects (font (size 1.27 1.27)) hide)
+    )
+    (property "Critical" "N" (id 4) (at 26.67 53.34 0)
+      (effects (font (size 1.27 1.27)) hide)
+    )
+    (property "Notes" "Bypass capacitor for PWR/GND coupling." (id 5) (at 26.67 53.34 0)
       (effects (font (size 1.27 1.27)) hide)
     )
@@
       (effects (font (size 1.27 1.27)) hide)
     )
+    (property "Critical" "N" (id 4) (at 39.37 133.35 0)
+      (effects (font (size 1.27 1.27)) hide)
+    )
+    (property "Notes" "Bypass capacitor for PWR/GND coupling." (id 5) (at 39.37 133.35 0)
+      (effects (font (size 1.27 1.27)) hide)
+    )
     (pin "1")
     (pin "2")
@@
       (effects (font (size 1.27 1.27)) hide)
     )
-    (property "Datasheet" "" (id 3) (at 233.68 39.37 0)
+    (property "Datasheet" "https://www.latticesemi.com/view_document?document_id=24635" (id 3) (at 233.68 39.37 0)
+      (effects (font (size 1.27 1.27)) hide)
+    )
+    (property "Critical" "Y" (id 4) (at 229.87 41.91 0)
+      (effects (font (size 1.27 1.27)) hide)
+    )
+    (property "Description" "FPGA - Field Programmable Gate Array 8K LUTs 86I/O Inst- on DSP 1.2V -5 Spd" (id 5) (at 229.87 41.91 0)
+      (effects (font (size 1.27 1.27)) hide)
+    )
+    (property "MFN" "Lattice" (id 6) (at 229.87 41.91 0)
+      (effects (font (size 1.27 1.27)) hide)
+    )
+    (property "MFP" "LFXP2-8E-5MN132C" (id 7) (at 229.87 41.91 0)
+      (effects (font (size 1.27 1.27)) hide)
+    )
+    (property "Notes" "FPGA used for the bulk of the cartridge's functions (MBC emulation, SPI bridge, MMU functions, etc.)." (id 8) (at 229.87 41.91 0)
+      (effects (font (size 1.27 1.27)) hide)
+    )
+    (property "Package ID" "CSBGA-132" (id 9) (at 229.87 41.91 0)
+      (effects (font (size 1.27 1.27)) hide)
+    )
+    (property "Source" "SPEC" (id 10) (at 229.87 41.91 0)
       (effects (font (size 1.27 1.27)) hide)
     )
@@
       (effects (font (size 1.27 1.27)) hide)
     )
+    (property "Critical" "N" (id 4) (at 52.07 156.21 0)
+      (effects (font (size 1.27 1.27)) hide)
+    )
+    (property "Notes" "Bypass capacitor for PWR/GND coupling." (id 5) (at 52.07 156.21 0)
+      (effects (font (size 1.27 1.27)) hide)
+    )
     (pin "1")
     (pin "2")
@@
       (effects (font (size 1.27 1.27)) hide)
     )
+    (property "Critical" "N" (id 4) (at 64.77 156.21 0)
+      (effects (font (size 1.27 1.27)) hide)
+    )
+    (property "Notes" "Bypass capacitor for PWR/GND coupling." (id 5) (at 64.77 156.21 0)
+      (effects (font (size 1.27 1.27)) hide)
+    )

Commit message: Added more symbol information
Parts:
- C19, C20, C21, C22, C23, C24, C25, C30, C31, C32: Source (none) -> ANY
- R15: Critical (none) -> Y; Source (none) -> ANY; Tolerance (none) -> 10%
Changed lines of the file:
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@@
+      (effects (font (size 1.27 1.27)) hide)
+    )
+    (property "Source" "ANY" (id 6) (at 204.47 29.21 0)
       (effects (font (size 1.27 1.27)) hide)
     )
@@
       (effects (font (size 1.27 1.27)) hide)
     )
+    (property "Source" "ANY" (id 6) (at 39.37 156.21 0)
+      (effects (font (size 1.27 1.27)) hide)
+    )
     (pin "1")
     (pin "2")
@@
       (effects (font (size 1.27 1.27)) hide)
     )
+    (property "Source" "ANY" (id 6) (at 116.84 36.83 0)
+      (effects (font (size 1.27 1.27)) hide)
+    )
     (pin "1")
     (pin "2")
@@
     )
     (property "Datasheet" "~" (id 3) (at 77.47 133.35 0)
+      (effects (font (size 1.27 1.27)) hide)
+    )
+    (property "Tolerance" "10%" (id 4) (at 77.47 133.35 0)
+      (effects (font (size 1.27 1.27)) hide)
+    )
+    (property "Source" "ANY" (id 5) (at 77.47 133.35 0)
+      (effects (font (size 1.27 1.27)) hide)
+    )
+    (property "Critical" "Y" (id 6) (at 77.47 133.35 0)
       (effects (font (size 1.27 1.27)) hide)
     )
@@
       (effects (font (size 1.27 1.27)) hide)
     )
+    (property "Source" "ANY" (id 6) (at 180.34 134.62 0)
+      (effects (font (size 1.27 1.27)) hide)
+    )
     (pin "1")
     (pin "2")
@@
     )
     (property "Notes" "Bypass capacitor for PWR/GND coupling." (id 5) (at 64.77 133.35 0)
+      (effects (font (size 1.27 1.27)) hide)
+    )
+    (property "Source" "ANY" (id 6) (at 64.77 133.35 0)
       (effects (font (size 1.27 1.27)) hide)
     )
@@
       (effects (font (size 1.27 1.27)) hide)
     )
+    (property "Source" "ANY" (id 6) (at 52.07 133.35 0)
+      (effects (font (size 1.27 1.27)) hide)
+    )
     (pin "1")
     (pin "2")
@@
     )
     (property "Notes" "Bypass capacitor for PWR/GND coupling." (id 5) (at 26.67 53.34 0)
+      (effects (font (size 1.27 1.27)) hide)
+    )
+    (property "Source" "ANY" (id 6) (at 26.67 53.34 0)
       (effects (font (size 1.27 1.27)) hide)
     )
@@
     )
     (property "Notes" "Bypass capacitor for PWR/GND coupling." (id 5) (at 39.37 133.35 0)
+      (effects (font (size 1.27 1.27)) hide)
+    )
+    (property "Source" "ANY" (id 6) (at 39.37 133.35 0)
       (effects (font (size 1.27 1.27)) hide)
     )
@@
       (effects (font (size 1.27 1.27)) hide)
     )
+    (property "Source" "ANY" (id 6) (at 52.07 156.21 0)
+      (effects (font (size 1.27 1.27)) hide)
+    )
     (pin "1")
     (pin "2")
@@
       (effects (font (size 1.27 1.27)) hide)
     )
+    (property "Source" "ANY" (id 6) (at 64.77 156.21 0)
+      (effects (font (size 1.27 1.27)) hide)
+    )

Commit message: Assigned and made a few footprints
Parts:
- C19, C20, C21, C22, C23, C24, C25, C30, C31, C32: footprint (none) -> Capacitor_SMD:C_0402_1005Metric_Pad0.74x0.62mm_HandSolder
- U9: footprint (none) -> SamacSys_Parts:BGA132C50P14X14_800X800X135
Changed lines of the file:
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@@
       (effects (font (size 1.27 1.27)) (justify left))
     )
-    (property "Footprint" "" (id 2) (at 205.4352 33.02 0)
+    (property "Footprint" "Capacitor_SMD:C_0402_1005Metric_Pad0.74x0.62mm_HandSolder" (id 2) (at 205.4352 33.02 0)
       (effects (font (size 1.27 1.27)) hide)
     )
@@
       (effects (font (size 1.27 1.27)) (justify left))
     )
-    (property "Footprint" "" (id 2) (at 101.6 121.92 0)
+    (property "Footprint" "SamacSys_Parts:BGA132C50P14X14_800X800X135" (id 2) (at 101.6 121.92 0)
       (effects (font (size 1.27 1.27)) hide)
     )
@@
       (effects (font (size 1.27 1.27)) (justify left))
     )
-    (property "Footprint" "" (id 2) (at 62.23 41.91 0)
+    (property "Footprint" "SamacSys_Parts:BGA132C50P14X14_800X800X135" (id 2) (at 62.23 41.91 0)
       (effects (font (size 1.27 1.27)) hide)
     )
@@
       (effects (font (size 1.27 1.27)) (justify left))
     )
-    (property "Footprint" "" (id 2) (at 152.4 25.4 0)
+    (property "Footprint" "SamacSys_Parts:BGA132C50P14X14_800X800X135" (id 2) (at 152.4 25.4 0)
       (effects (font (size 1.27 1.27)) hide)
     )
@@
       (effects (font (size 1.27 1.27)) (justify left))
     )
-    (property "Footprint" "" (id 2) (at 40.3352 160.02 0)
+    (property "Footprint" "Capacitor_SMD:C_0402_1005Metric_Pad0.74x0.62mm_HandSolder" (id 2) (at 40.3352 160.02 0)
       (effects (font (size 1.27 1.27)) hide)
     )
@@
       (effects (font (size 1.27 1.27)) (justify left))
     )
-    (property "Footprint" "" (id 2) (at 117.8052 40.64 0)
+    (property "Footprint" "Capacitor_SMD:C_0402_1005Metric_Pad0.74x0.62mm_HandSolder" (id 2) (at 117.8052 40.64 0)
       (effects (font (size 1.27 1.27)) hide)
     )
@@
       (effects (font (size 1.27 1.27)) (justify left))
     )
-    (property "Footprint" "" (id 2) (at 181.3052 138.43 0)
+    (property "Footprint" "Capacitor_SMD:C_0402_1005Metric_Pad0.74x0.62mm_HandSolder" (id 2) (at 181.3052 138.43 0)
       (effects (font (size 1.27 1.27)) hide)
     )
@@
       (effects (font (size 1.27 1.27)) (justify left))
     )
-    (property "Footprint" "" (id 2) (at 65.7352 137.16 0)
+    (property "Footprint" "Capacitor_SMD:C_0402_1005Metric_Pad0.74x0.62mm_HandSolder" (id 2) (at 65.7352 137.16 0)
       (effects (font (size 1.27 1.27)) hide)
     )
@@
       (effects (font (size 1.27 1.27)) (justify left))
     )
-    (property "Footprint" "" (id 2) (at 218.44 123.19 0)
+    (property "Footprint" "SamacSys_Parts:BGA132C50P14X14_800X800X135" (id 2) (at 218.44 123.19 0)
       (effects (font (size 1.27 1.27)) hide)
     )
@@
       (effects (font (size 1.27 1.27)) (justify left))
     )
-    (property "Footprint" "" (id 2) (at 53.0352 137.16 0)
+    (property "Footprint" "Capacitor_SMD:C_0402_1005Metric_Pad0.74x0.62mm_HandSolder" (id 2) (at 53.0352 137.16 0)
       (effects (font (size 1.27 1.27)) hide)
     )
@@
       (effects (font (size 1.27 1.27)) (justify left))
     )
-    (property "Footprint" "" (id 2) (at 27.6352 57.15 0)
+    (property "Footprint" "Capacitor_SMD:C_0402_1005Metric_Pad0.74x0.62mm_HandSolder" (id 2) (at 27.6352 57.15 0)
       (effects (font (size 1.27 1.27)) hide)
     )
@@
       (effects (font (size 1.27 1.27)) (justify left))
     )
-    (property "Footprint" "" (id 2) (at 40.3352 137.16 0)
+    (property "Footprint" "Capacitor_SMD:C_0402_1005Metric_Pad0.74x0.62mm_HandSolder" (id 2) (at 40.3352 137.16 0)
       (effects (font (size 1.27 1.27)) hide)
     )
@@
       (effects (font (size 1.27 1.27)) (justify left))
     )
-    (property "Footprint" "" (id 2) (at 233.68 39.37 0)
+    (property "Footprint" "SamacSys_Parts:BGA132C50P14X14_800X800X135" (id 2) (at 233.68 39.37 0)
       (effects (font (size 1.27 1.27)) hide)
     )
@@
       (effects (font (size 1.27 1.27)) (justify left))
     )
-    (property "Footprint" "" (id 2) (at 53.0352 160.02 0)
+    (property "Footprint" "Capacitor_SMD:C_0402_1005Metric_Pad0.74x0.62mm_HandSolder" (id 2) (at 53.0352 160.02 0)
       (effects (font (size 1.27 1.27)) hide)
     )
@@
       (effects (font (size 1.27 1.27)) (justify left))
     )
-    (property "Footprint" "" (id 2) (at 65.7352 160.02 0)
-      (effects (font (size 1.27 1.27)) hide)
-    )
+    (property "Footprint" "Capacitor_SMD:C_0402_1005Metric_Pad0.74x0.62mm_HandSolder" (id 2) (at 65.7352 160.02 0)
+      (effects (font (size 1.27 1.27)) hide)
+    )
