File: CartGen4/bus-transceivers.kicad_sch (KiCad schematic)
At the start: 5 parts, among them U4 NXS0108BQX, U6 NXS0108BQX, U7 NXS0108BQX, U8 NXS0104BQX

Commit message: Added more symbol information
Parts:
- R14: Critical (none) -> Y; Source (none) -> ANY; Tolerance (none) -> 10%
Changed lines of the file:
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@@
+      (effects (font (size 1.27 1.27)) hide)
+    )
+    (property "Tolerance" "10%" (id 4) (at 49.53 73.66 0)
+      (effects (font (size 1.27 1.27)) hide)
+    )
+    (property "Source" "ANY" (id 5) (at 49.53 73.66 0)
+      (effects (font (size 1.27 1.27)) hide)
+    )
+    (property "Critical" "Y" (id 6) (at 49.53 73.66 0)
       (effects (font (size 1.27 1.27)) hide)
     )

Commit message: Assigned and made a few footprints
Parts:
- U4, U6, U7: footprint (none) -> SamacSys_Parts:NXS0108BQX
- U8: footprint (none) -> SamacSys_Parts:NXS0104BQX
Changed lines of the file:
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@@
       (effects (font (size 1.27 1.27)) (justify left))
     )
-    (property "Footprint" "" (id 2) (at 129.54 90.17 90)
+    (property "Footprint" "SamacSys_Parts:NXS0108BQX" (id 2) (at 129.54 90.17 90)
       (effects (font (size 1.27 1.27)) hide)
     )
@@
       (effects (font (size 1.27 1.27)) (justify left))
     )
-    (property "Footprint" "" (id 2) (at 129.54 149.86 90)
+    (property "Footprint" "SamacSys_Parts:NXS0108BQX" (id 2) (at 129.54 149.86 90)
       (effects (font (size 1.27 1.27)) hide)
     )
@@
       (effects (font (size 1.27 1.27)) (justify left))
     )
-    (property "Footprint" "" (id 2) (at 129.54 31.75 90)
+    (property "Footprint" "SamacSys_Parts:NXS0108BQX" (id 2) (at 129.54 31.75 90)
       (effects (font (size 1.27 1.27)) hide)
     )
@@
       (effects (font (size 1.27 1.27)) (justify left))
     )
-    (property "Footprint" "" (id 2) (at 241.3 97.79 90)
-      (effects (font (size 1.27 1.27)) hide)
-    )
+    (property "Footprint" "SamacSys_Parts:NXS0104BQX" (id 2) (at 241.3 97.79 90)
+      (effects (font (size 1.27 1.27)) hide)
+    )

Commit message: Assigned all footprints
Parts:
- R14: footprint (none) -> Resistor_SMD:R_0603_1608Metric_Pad0.98x0.95mm_HandSolder
Changed lines of the file:
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@@
       (effects (font (size 1.27 1.27)) (justify left))
     )
-    (property "Footprint" "" (id 2) (at 47.752 73.66 90)
+    (property "Footprint" "Resistor_SMD:R_0603_1608Metric_Pad0.98x0.95mm_HandSolder" (id 2) (at 47.752 73.66 90)
       (effects (font (size 1.27 1.27)) hide)
     )
