File: CartGen4/gb_reset_clock.kicad_sch (KiCad schematic)
At the start: 7 parts, among them SW1 SW_Push, U2 SN74LV1T34DCKR, U3 SIT8008BI-73-33E-33.333333G

Commit message: Added more symbol information
Parts:
- C18: Source (none) -> ANY
- D1: MFN (none) -> Nexperia; MFP (none) -> PESD3V3Y1BSFYL; Notes ESD protection for exposed reset button. -> ESD protection for exposed reset button. Must have a clampi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; Package ID (none) -> DSN-0603-2; Source (none) -> ANY; Voltage (none) -> 3.3V
- R11, R13: Critical (none) -> Y; Source (none) -> ANY; Tolerance (none) -> 10%
- SW1: Critical (none) -> Y
Changed lines of the file:
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@@
       (effects (font (size 1.27 1.27)) hide)
     )
-    (property "Notes" "ESD protection for exposed reset button." (id 5) (at 199.39 72.39 0)
+    (property "Notes" "ESD protection for exposed reset button. Must have a clamping voltage no larger than 3.75V." (id 5) (at 199.39 72.39 0)
+      (effects (font (size 1.27 1.27)) hide)
+    )
+    (property "Description" "ESD Suppressors / TVS Diodes PESD3V3Y1BSF/SOD962/SOD962" (id 6) (at 199.39 72.39 0)
+      (effects (font (size 1.27 1.27)) hide)
+    )
+    (property "MFN" "Nexperia" (id 7) (at 199.39 72.39 0)
+      (effects (font (size 1.27 1.27)) hide)
+    )
+    (property "MFP" "PESD3V3Y1BSFYL" (id 8) (at 199.39 72.39 0)
+      (effects (font (size 1.27 1.27)) hide)
+    )
+    (property "Package ID" "DSN-0603-2" (id 9) (at 199.39 72.39 0)
+      (effects (font (size 1.27 1.27)) hide)
+    )
+    (property "Source" "ANY" (id 10) (at 199.39 72.39 0)
+      (effects (font (size 1.27 1.27)) hide)
+    )
+    (property "Voltage" "3.3V" (id 11) (at 199.39 72.39 0)
       (effects (font (size 1.27 1.27)) hide)
     )
@@
     )
     (property "Datasheet" "~" (id 3) (at 57.15 60.96 0)
+      (effects (font (size 1.27 1.27)) hide)
+    )
+    (property "Tolerance" "10%" (id 4) (at 57.15 60.96 0)
+      (effects (font (size 1.27 1.27)) hide)
+    )
+    (property "Source" "ANY" (id 5) (at 57.15 60.96 0)
+      (effects (font (size 1.27 1.27)) hide)
+    )
+    (property "Critical" "Y" (id 6) (at 57.15 60.96 0)
       (effects (font (size 1.27 1.27)) hide)
     )
@@
       (effects (font (size 1.27 1.27)) hide)
     )
+    (property "Critical" "Y" (id 4) (at 189.23 66.04 0)
+      (effects (font (size 1.27 1.27)) hide)
+    )
     (pin "1")
     (pin "2")
@@
       (effects (font (size 1.27 1.27)) hide)
     )
+    (property "Source" "ANY" (id 6) (at 111.76 69.85 0)
+      (effects (font (size 1.27 1.27)) hide)
+    )
     (pin "1")
     (pin "2")
@@
       (effects (font (size 1.27 1.27)) hide)
     )
+    (property "Tolerance" "10%" (id 4) (at 52.07 127 0)
+      (effects (font (size 1.27 1.27)) hide)
+    )
+    (property "Source" "ANY" (id 5) (at 52.07 127 0)
+      (effects (font (size 1.27 1.27)) hide)
+    )
+    (property "Critical" "Y" (id 6) (at 52.07 127 0)
+      (effects (font (size 1.27 1.27)) hide)
+    )

Commit message: Converted footprints
Parts:
- U2: footprint SOT65P210X110-5N -> SamacSys_Parts:SOT65P210X110-5N
Changed lines of the file:
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@@
     (property "Reference" "U2" (id 0) (at 78.74 110.49 0))
     (property "Value" "SN74LV1T34DCKR" (id 1) (at 78.74 113.03 0))
-    (property "Footprint" "SOT65P210X110-5N" (id 2) (at 87.63 115.57 0)
+    (property "Footprint" "SamacSys_Parts:SOT65P210X110-5N" (id 2) (at 87.63 115.57 0)
       (effects (font (size 1.27 1.27)) (justify left) hide)
     )

Commit message: Made and assigned clock footprint
Parts:
- U3: footprint (none) -> SamacSys_Parts:SIT8008BI-73-33E-33.333333G
Changed lines of the file:
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@@
     (property "Reference" "U3" (id 0) (at 78.74 53.34 0))
     (property "Value" "SIT8008BI-73-33E-33.333333G" (id 1) (at 80.01 55.88 0))
-    (property "Footprint" "" (id 2) (at 72.39 58.42 0)
+    (property "Footprint" "SamacSys_Parts:SIT8008BI-73-33E-33.333333G" (id 2) (at 72.39 58.42 0)
       (effects (font (size 1.27 1.27)) hide)
     )

Commit message: Assigned and made a few footprints
Parts:
- C18: footprint (none) -> Capacitor_SMD:C_0402_1005Metric_Pad0.74x0.62mm_HandSolder
Changed lines of the file:
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@@
       (effects (font (size 1.27 1.27)) (justify left))
     )
-    (property "Footprint" "" (id 2) (at 112.7252 73.66 0)
+    (property "Footprint" "Capacitor_SMD:C_0402_1005Metric_Pad0.74x0.62mm_HandSolder" (id 2) (at 112.7252 73.66 0)
       (effects (font (size 1.27 1.27)) hide)
     )

Commit message: Assigned all footprints
Parts:
- C18: footprint Capacitor_SMD:C_0402_1005Metric_Pad0.74x0.62mm_HandSolder -> Capacitor_SMD:C_0603_1608Metric_Pad1.08x0.95mm_HandSolder
- D1: footprint (none) -> SamacSys_Parts:PESD3V3Y1BSFYL
- R11, R13: footprint (none) -> Resistor_SMD:R_0603_1608Metric_Pad0.98x0.95mm_HandSolder
- SW1: footprint (none) -> Button_Switch_SMD:SW_SPST_TL3305A
Changed lines of the file:
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@@
       (effects (font (size 1.27 1.27)) (justify right))
     )
-    (property "Footprint" "" (id 2) (at 199.39 72.39 0)
+    (property "Footprint" "SamacSys_Parts:PESD3V3Y1BSFYL" (id 2) (at 199.39 72.39 0)
       (effects (font (size 1.27 1.27)) hide)
     )
@@
     (property "Reference" "R13" (id 0) (at 57.15 54.61 90))
     (property "Value" "1K" (id 1) (at 57.15 57.15 90))
-    (property "Footprint" "" (id 2) (at 57.15 62.738 90)
+    (property "Footprint" "Resistor_SMD:R_0603_1608Metric_Pad0.98x0.95mm_HandSolder" (id 2) (at 57.15 62.738 90)
       (effects (font (size 1.27 1.27)) hide)
     )
@@
     (property "Reference" "SW1" (id 0) (at 189.23 58.42 0))
     (property "Value" "SW_Push" (id 1) (at 189.23 60.96 0))
-    (property "Footprint" "" (id 2) (at 189.23 60.96 0)
+    (property "Footprint" "Button_Switch_SMD:SW_SPST_TL3305A" (id 2) (at 189.23 60.96 0)
       (effects (font (size 1.27 1.27)) hide)
     )
@@
       (effects (font (size 1.27 1.27)) (justify left))
     )
-    (property "Footprint" "Capacitor_SMD:C_0402_1005Metric_Pad0.74x0.62mm_HandSolder" (id 2) (at 112.7252 73.66 0)
+    (property "Footprint" "Capacitor_SMD:C_0603_1608Metric_Pad1.08x0.95mm_HandSolder" (id 2) (at 112.7252 73.66 0)
       (effects (font (size 1.27 1.27)) hide)
     )
@@
       (effects (font (size 1.27 1.27)) (justify right))
     )
-    (property "Footprint" "" (id 2) (at 53.848 127 90)
-      (effects (font (size 1.27 1.27)) hide)
-    )
+    (property "Footprint" "Resistor_SMD:R_0603_1608Metric_Pad0.98x0.95mm_HandSolder" (id 2) (at 53.848 127 90)
+      (effects (font (size 1.27 1.27)) hide)
+    )
